Commit message: Full model of wheelchair. Updated the launchers

File: model/wheelchair.urdf (robot description, URDF)
Before this commit: robot wheelchair, 14 links, 13 joints
Links:
- removed link platform_link
- added link platformdown_link; visual box size=0.4 0.51 0.031
- added link platformup_link; visual box size=0.5 0.51 0.031
- added link sonar_0xe4_link; visual box size=0.012 0.032 0.015
- added link sonar_0xe6_link; visual box size=0.012 0.032 0.015
- added link sonar_0xe8_link; visual box size=0.012 0.032 0.015
- added link sonar_0xee_link; visual box size=0.012 0.032 0.015
- added link sonar_0xf0_link; visual box size=0.012 0.032 0.015
- added link sonar_0xf2_link; visual box size=0.012 0.032 0.015
- link backseat_link: geometry visual box size=0.12 0.51 0.83
- link base_link: geometry collision box size=1.1 0.80 1.4; visual box size=0.63 0.31 0.35
- link seat_link: geometry visual box size=0.48 0.51 0.12
- link sonar_0xe0_link: geometry visual box size=0.012 0.032 0.015
- link sonar_0xe2_link: geometry visual box size=0.012 0.032 0.015
- link sonar_0xea_link: geometry visual box size=0.012 0.032 0.015
- link sonar_0xec_link: geometry visual box size=0.012 0.032 0.015
Joints:
- removed joint platform_joint
- added joint platformdown_joint: type fixed, parent seat_link, child platformdown_link, origin xyz=-0.4 0.0 -0.0445 rpy=0.0 0 0
- added joint platformup_joint: type fixed, parent seat_link, child platformup_link, origin xyz=-0.45 0.0 0.1 rpy=0.0 0 0
- added joint sonar_0xe4_joint: type fixed, parent base_link, child sonar_0xe4_link, origin xyz=-0.165 -0.265 0.205 rpy=0 0 -1.5705
- added joint sonar_0xe6_joint: type fixed, parent base_link, child sonar_0xe6_link, origin xyz=-0.513 -0.265 0.2455 rpy=0 0 -1.5705
- added joint sonar_0xe8_joint: type fixed, parent base_link, child sonar_0xe8_link, origin xyz=-0.62 -0.238 0.3975 rpy=0 0 -3.141
- added joint sonar_0xee_joint: type fixed, parent base_link, child sonar_0xee_link, origin xyz=-0.165 0.265 0.205 rpy=0 0 1.5705
- added joint sonar_0xf0_joint: type fixed, parent base_link, child sonar_0xf0_link, origin xyz=-0.513 0.265 0.2455 rpy=0 0 1.5705
- added joint sonar_0xf2_joint: type fixed, parent base_link, child sonar_0xf2_link, origin xyz=-0.62 0.238 0.3975 rpy=0 0 -3.141
- joint backseat_joint: origin xyz=0.0 -0.30 0.355 rpy=0.3 0 0 -> xyz=-0.30 0.0 0.355 rpy=0 -0.3 0
- joint backwheel0_joint: axis (none) -> 0 1 0; origin xyz=-0.225 -0.405 -0.18 rpy=0 0 0 -> xyz=-0.405 -0.225 -0.17 rpy=0 0 0; type fixed -> continuous
- joint backwheel1_joint: axis (none) -> 0 1 0; origin xyz=0.225 -0.405 -0.18 rpy=0 0 0 -> xyz=-0.405 0.225 -0.17 rpy=0 0 0; type fixed -> continuous
- joint frontwheel0_joint: axis (none) -> 0 1 0; origin xyz=-0.285 0.385 -0.18 rpy=0 0 0 -> xyz=0.385 -0.285 -0.17 rpy=0 0 0; type fixed -> continuous
- joint frontwheel1_joint: axis (none) -> 0 1 0; origin xyz=0.285 0.385 -0.18 rpy=0 0 0 -> xyz=0.385 0.285 -0.17 rpy=0 0 0; type fixed -> continuous
- joint seat_joint: axis (none) -> 0 0 1; limit (none) -> lower=0.0 upper=0.15 effort=1000.0 velocity=0.01; origin xyz=0.0 0.075 0.2975 rpy=0 0 0 -> xyz=0.075 0.0 0.2975 rpy=0 0 0; type fixed -> prismatic
- joint sonar_0xe0_joint: origin xyz=0.10 0.565 -0.05 -> xyz=0.565 -0.10 -0.05
- joint sonar_0xe2_joint: origin xyz=0.265 0.385 0.01 rpy=0 0 0 -> xyz=0.385 -0.265 0.01 rpy=0 0 0
- joint sonar_0xea_joint: origin xyz=-0.10 0.565 -0.05 -> xyz=0.565 0.10 -0.05
- joint sonar_0xec_joint: origin xyz=-0.265 0.385 0.01 rpy=0 0 0 -> xyz=0.385 0.265 0.01 rpy=0 0 0
- joint wheel0_joint: axis (none) -> 0 1 0; origin xyz=-0.295 0.095 -0.085 rpy=0 0 0 -> xyz=0.095 -0.295 -0.085 rpy=0 0 0; type fixed -> continuous
- joint wheel1_joint: axis (none) -> 0 1 0; origin xyz=0.295 0.095 -0.085 rpy=0 0 0 -> xyz=0.095 0.295 -0.085 rpy=0 0 0; type fixed -> continuous

Commit message: Kinect stuff, still not proeprly working

File: model/wheelchair.urdf (robot description, URDF)
Before this commit: robot wheelchair, 21 links, 20 joints
Links:
- added link camera_link; visual box size=0.12 0.32 0.15
Joints:
- added joint camera_joint: type fixed, parent base_link, child camera_link, origin xyz=0.565 -0.00 0.2975

Commit message: Fixed position of the front sonars

File: model/wheelchair.urdf (robot description, URDF)
Before this commit: robot wheelchair, 22 links, 21 joints
Joints:
- joint sonar_0xe0_joint: origin xyz=0.565 -0.10 -0.05 -> xyz=0.365 -0.10 -0.05
- joint sonar_0xea_joint: origin xyz=0.565 0.10 -0.05 -> xyz=0.365 0.10 -0.05
